File: hardware/sensorboard_spectrometer_rev0.kicad_pcb (KiCad board)
At the start: 2 copper layers, 69.1 x 54.9 mm, 41 parts, among them IC1 CAT4101, U1 MICROSPEC-C12666MA, U10 ADS1115IDGS, U11 TPS61088RHLT, U4 W25Q16JVSS, U5 TLV9001IDCK, U6 MCP9808_MSOP, U7 TRANSLATOR-TXS0108E, U8 DS3231MZ, U9 LT3045xDD

Commit message: pcb
Parts:
- L1, L2: footprint Inductor_SMD:L_0805_2012Metric -> Inductor_SMD:L_0603_1608Metric
- U3: value ~ -> LILTGO touch
- moved C2 0.60 mm to (49.7, 39.3)
- moved L1 0.27 mm to (51.5, 39.3)
Routing:
- net 5V: track 120.6 -> 121.2 mm
