File: hardware/sensorboard_spectrometer_rev0.kicad_sch (KiCad schematic)
At the start: 27 parts, among them J4 USB_C_Programming, Q1 BC817, Q2 BC817, SW1 RESET, U1 MICROSPEC-C12666MA, U2 AD7940, U3 OPA344, U4 ESP32-S3-WROOM-1-N8, U6 CP2102N-Axx-xQFN24, U8 DS3231MZ

Commit message: Add Lilygo and the rest of the components
Parts:
- removed C17, C18: 220uF, Capacitor_Tantalum_SMD:CP_EIA-3528-21_Kemet-B, symbol Device:C_Polarized
- removed C3: C_Polarized 100uF, Capacitor_Tantalum_SMD:CP_EIA-3528-21_Kemet-B, symbol Device:C_Polarized
- removed C9: 100 nF, Capacitor_SMD:C_0805_2012Metric, symbol Device:C
- removed J4: USB_C_Programming, footprint:USB_C_Receptacle_HRO_TYPE-C-31-M-12, symbol Connector:USB_C_Receptacle_USB2.0
- removed Q1, Q2: BC817, Package_TO_SOT_SMD:SOT-23, symbol Transistor_BJT:BC817
- removed R10, R9: 4.7K, Resistor_SMD:R_0603_1608Metric, symbol Device:R
- removed R15, R16: 5.1K, Resistor_SMD:R_0603_1608Metric, symbol Device:R_Small
- removed SW1: RESET, footprint:Alps_SKRK, symbol Switch:SW_Push
- removed TP3: 32Khz, TestPoint:TestPoint_Pad_D1.5mm, symbol Connector:TestPoint
- removed U3: OPA344, sensorboard_spectrometer_rev0:SOT23-5, symbol sensorboard_spectrometer_rev0-eagle-import:OPA344
- removed U4: ESP32-S3-WROOM-1-N8, footprint:ESP32-S3-WROOM-1-N8, symbol ESP32-S3-WROOM-1-N8:ESP32-S3-WROOM-1-N8
- removed U6: CP2102N-Axx-xQFN24, Package_DFN_QFN:QFN-24-1EP_4x4mm_P0.5mm_EP2.6x2.6mm, symbol Interface_USB:CP2102N-Axx-xQFN24
- added BAT_IN, BAT_OU_LILYGO: M02-JST-2MM-SMT, motherboard_rev0:JST-2-SMD, symbol motherboard_rev0-eagle-import:M02-JST-2MM-SMT
- added BT1: Battery_Cell, symbol Device:Battery_Cell
- added C3, C4, C7, C8, C9: 0.1uF, sensorboard_spectrometer_rev0:0603, symbol sensorboard_spectrometer_rev0-eagle-import:notes_mark5_CAP0603
- added C5, C6: 220uF, sensorboard_spectrometer_rev0:0603, symbol sensorboard_spectrometer_rev0-eagle-import:notes_mark5_CAP0603
- added D1: LED, symbol Device:LED
- added IC1: CAT4101, F9ZYROSHVXBZZL3:TO263_5, symbol F9ZYROSHVXBZZL3-eagle-import:CAT4101
- added L2: 4.7uH, sensorboard_spectrometer_rev0:0805, symbol sensorboard_spectrometer_rev0-eagle-import:INDUCTOR0805
- added R10, R11: 4.7 K, Resistor_SMD:R_0603_1608Metric, symbol Device:R_Small
- added R2: 10 K, Resistor_SMD:R_0603_1608Metric, symbol Device:R_Small
- added R4: 22.1 K, Resistor_SMD:R_0603_1608Metric, symbol Device:R_Small
- added R5: 5K, F9ZYROSHVXBZZL3:RTRIM64W, symbol F9ZYROSHVXBZZL3-eagle-import:R-TRIMM64W
- added R6: 500, Resistor_SMD:R_0603_1608Metric, symbol Device:R_Small
- added R7: 56.2 K, Resistor_SMD:R_0603_1608Metric, symbol Device:R_Small
- added R9: 40 K, Resistor_SMD:R_0603_1608Metric, symbol Device:R_Small
- added U$5: SWITCH_SPDT, motherboard_rev0:KPS-1290, symbol motherboard_rev0-eagle-import:SWITCH_SPDT
- added U11: TPS61088RHLT, TPS61088RHLT:IC_MSP430FR2522IRHLR, symbol TPS61088RHLT:TPS61088RHLT
- added U3: ~, symbol micross:lilugo-touch_1.9{dblquote}
- added U4: W25Q16JVSS, Package_SO:SOIC-8_5.3x5.3mm_P1.27mm, symbol Memory_Flash:W25Q16JVSS
- added U5: TLV9001IDCK, Package_TO_SOT_SMD:SOT-353_SC-70-5, symbol Amplifier_Operational:TLV9001IDCK
- added U6: MCP9808_MSOP, Package_SO:MSOP-8_3x3mm_P0.65mm, symbol Sensor_Temperature:MCP9808_MSOP
- added U7: TRANSLATOR-TXS0108E, sensorboard_spectrometer_rev0:TSSOP-20, symbol sensorboard_spectrometer_rev0-eagle-import:TRANSLATOR-TXS0108E
- added U9: LT3045xDD, Package_DFN_QFN:DFN-10-1EP_3x3mm_P0.5mm_EP1.65x2.38mm, symbol Regulator_Linear:LT3045xDD
- R3: value 10 K -> 100 K
- R8: value 10 K -> 40 K
Connections:
- net +3V3: now also C4.1, R10.1, R11.1, U3.12 (3V3), U3.13 (3V3); no longer R3.1
- net 5V: now also C7.1, IC1.2 (VIN), U3.24 (5V), U7.19 (VCCB), U9.10 (OUT)
- net CLK_5V: now also U7.15 (B5), U7.6 (A5)
- net EOS_5V: now also U7.14 (B6), U7.7 (A6)
- net GAIN_5V: now also U7.13 (B7)
- net GND: now also R3.2, R8.2, BAT_IN.1 (2), BAT_OU_LILYGO.1 (2), BT1.2 (-), C3.2, C4.2, C5.2, C6.1, C7.2, C9.2, D1.1 (K), IC1.3 (GND), IC1.TAB, R4.1, R5.1 (A), U11.10 (SS), U11.13 (MODE), U11.20 (AGND), U11.21 (PGND), U3.1 (GND), U3.10 (GND), U3.11 (GND), U3.2 (GND), U3.23 (GND), U4.4 (GND), U5.2 (V-), U6.4 (GND), U6.5 (A2), U6.6 (A1), U6.7 (A0), U7.11 (GND), U9.11 (GND), U9.5 (ILIM), U9.6 (PGFB), U9.8 (GND)
- net I2C_SCL: now also R10.2, U3.6 (GPIO17), U6.2 (SCL)
- net I2C_SDA: now also R11.2, U3.5 (GPIO18), U6.1 (SDA)
- net SPI_CLK_5V: now also U7.16 (B4)
- net SPI_CS_5V: now also U7.18 (B2)
- net SPI_MISO_5V: now also U7.17 (B3)
- net ST_5V: now also U7.12 (B8)
- net V_SPEC: now also U5.5 (V+)
- net +BATT: now reaches D4.1 (K), U8.6 (VBAT)
- net +BATT: now also BT1.1 (+), C5.1, C6.2
- net at R1.2: now also U4.7 (~{HOLD}/~{RESET}/IO_{3})
- net at U2.3 (AN_IN): now also U5.1 (+), U5.4
- net at U1.2 (VIDEO): now also U5.3 (-)
- net DTR renamed 3.3V
- net 3.3V: now also C3.1, R2.1, U4.8 (VCC), U7.10 (OE), U7.2 (VCCA)
- net IO_2: no longer names the net of R12.2, U8.3 (~{INT}/SQW)
- net RTS: no longer names the net of R8.1
- net RTS: now also U11.19 (ILIM)
- new net: R2.2, U4.3 (~{WP}/IO_{2})
- new net: L2.2, R9.1, U11.4 (SW), U11.5 (SW), U11.6 (SW), U11.7 (SW)
- new net: C9.1, U11.1 (VCC)
- new net: R9.2, U11.3 (FSW)
- new net: R4.2, R7.2, U11.17 (FB)
- new net: C8.2, U11.8 (BOOT)
- new net: IC1.4 (RSET), R6.2
- new net: D1.2 (A), IC1.5 (LED)
- new net: R5.2 (S), R5.3 (E), R6.1
- new net: U11.11 (NC), U11.12 (NC)
- new net +3.7V: BAT_OU_LILYGO.2 (1), U$5.P, U11.9 (VIN)
- new net +3.7V_0: BAT_IN.2 (1), R3.1, U$5.O
- new net +5.5V: C8.1, L2.1, R7.1, U11.14 (VOUT), U11.15 (VOUT), U11.16 (VOUT), U11.2 (EN), U9.1 (IN), U9.2 (IN), U9.3 (EN/UV)
- new net GAIN_3V: U7.8 (A7)
- new net PWM_LED: IC1.1 (EN/PWM), U3.14 (GPIO1)
- new net SPI_CLK_3V: U3.19 (GPIO12), U4.6 (CLK), U7.5 (A4)
- new net SPI_CS_1_3V: U3.16 (GPIO3), U4.1 (~{CS})
- new net SPI_CS_3V: U3.17 (GPIO10), U7.3 (A2)
- new net SPI_MISO_3V: U3.20 (GPIO13), U4.2 (DO/IO_{1}), U7.4 (A3)
- new net SPI_MOSI_3V: U3.18 (GPIO11), U4.5 (DI/IO_{0})
- new net ST_3V: U7.9 (A8)
- no-connect marks 14 -> 8
Other:
- note added: "POWER SWITCH"
- note removed: "35,36,37 used by PSRAM"
- note removed: "INT to C3>"
- note removed: "RESET"
- moved on the sheet: C1, C2, D4, L1, R12, U1, U2, U8

Commit message: pcb
Parts:
- removed C5, C6: 220uF, sensorboard_spectrometer_rev0:0603, symbol sensorboard_spectrometer_rev0-eagle-import:notes_mark5_CAP0603
- removed D4: 1N5819WS, Diode_SMD:D_SOD-323, symbol Diode:MBR0530
- removed U$5: SWITCH_SPDT, motherboard_rev0:KPS-1290, symbol motherboard_rev0-eagle-import:SWITCH_SPDT
- removed U2: AD7940, sensorboard_spectrometer_rev0:SOT-23-6L, symbol sensorboard_spectrometer_rev0-eagle-import:AD7940
- added C10: 0.1uF, Capacitor_SMD:C_0603_1608Metric, symbol sensorboard_spectrometer_rev0-eagle-import:notes_mark5_CAP0603
- added R13, R14, R15: 0, Resistor_SMD:R_0603_1608Metric, symbol Device:R
- added SWITCH_SPDT1: M02-JST-2MM-SMT, Connector_JST:JST_EH_S2B-EH_1x02_P2.50mm_Horizontal, symbol motherboard_rev0-eagle-import:M02-JST-2MM-SMT
- added U10: ADS1115IDGS, Package_SO:TSSOP-10_3x3mm_P0.5mm, symbol Analog_ADC:ADS1115IDGS
- BAT_IN1: renamed from BAT_IN; footprint motherboard_rev0:JST-2-SMD -> Connector_JST:JST_EH_S2B-EH_1x02_P2.50mm_Horizontal
- BAT_OU_LILYGO1: renamed from BAT_OU_LILYGO; footprint motherboard_rev0:JST-2-SMD -> Connector_JST:JST_EH_S2B-EH_1x02_P2.50mm_Horizontal
- BT1: footprint (none) -> Battery:BatteryHolder_Keystone_1058_1x2032
- C1, C2, C3, C4, C7, C8, C9: footprint sensorboard_spectrometer_rev0:0603 -> Capacitor_SMD:C_0603_1608Metric
- D1: footprint (none) -> Connector_JST:JST_EH_S2B-EH_1x02_P2.50mm_Horizontal
- IC1: footprint F9ZYROSHVXBZZL3:TO263_5 -> Package_TO_SOT_SMD:TO-263-5_TabPin6
- L1, L2: footprint sensorboard_spectrometer_rev0:0805 -> Inductor_SMD:L_0805_2012Metric
- R5: footprint F9ZYROSHVXBZZL3:RTRIM64W -> Potentiometer_THT:Potentiometer_Runtron_RM-065_Vertical
- U1: footprint sensorboard_spectrometer_rev0:C12666MA -> mioss:C12880MA
- U11: footprint TPS61088RHLT:IC_MSP430FR2522IRHLR -> mioss:IC_MSP430FR2522IRHLR
- U3: footprint (none) -> micross:Untitled
- U7: footprint sensorboard_spectrometer_rev0:TSSOP-20 -> Package_SO:TSSOP-20_4.4x5mm_P0.5mm
Connections:
- net +3.7V: now also SWITCH_SPDT1.1 (2)
- net +3.7V_0: now also SWITCH_SPDT1.2 (1)
- net +3V3: now also C3.1, R1.1, R2.1, U4.8 (VCC), U6.8 (V_{DD}), C10.1, R13.1, R14.2, U10.8 (VDD); no longer U3.13 (3V3)
- net 3.3V: no longer C3.1, R1.1, R2.1, U4.8 (VCC), U7.2 (VCCA)
- net CLK_5V: no longer U7.6 (A5)
- net EOS_5V: no longer U7.7 (A6)
- net GND: now also C10.2, U10.1 (ADDR), U10.3 (GND)
- net I2C_SCL: now also U7.5 (A4)
- net I2C_SDA: now also U7.4 (A3)
- net SPI_CLK_3V: no longer U7.5 (A4)
- net SPI_CS_1_3V: now also R15.1; no longer U3.16 (GPIO3)
- net SPI_MISO_3V: no longer U7.4 (A3)
- net at U5.1 (+), U5.4: now also U10.4 (AIN0)
- net SPI_CLK_5V renamed I2C_SCL_5V
- net I2C_SCL_5V: now also U10.10 (SCL)
- net SPI_CS_3V: no longer names the net of U3.17 (GPIO10)
- net SPI_CS_3V: now also R15.2; no longer U7.3 (A2)
- net SPI_CS_5V: no longer names the net of U7.18 (B2)
- net SPI_MISO_5V renamed I2C_SDA_5V
- net I2C_SDA_5V: now also U10.9 (SDA)
- new net: R14.1, U3.13 (3V3)
- new net: R13.2, U7.2 (VCCA)
- new net CLK_3V: U7.6 (A5)
- new net EOS_3V: U7.7 (A6)
- no-connect marks 8 -> 11

Commit message: pcb
Parts:
- C1, C2: MP (none) -> C0603C223K5RACTU
- C10, C3, C4, C7, C8, C9: MP (none) -> C0603C104K3RACTU
- L1: footprint Inductor_SMD:L_0805_2012Metric -> Inductor_SMD:L_0603_1608Metric; MP (none) -> LQW18ASR10G00D
- L2: footprint Inductor_SMD:L_0805_2012Metric -> Inductor_SMD:L_0603_1608Metric; MP (none) -> LQW18AS4N7G00D
- R1, R12, R2: MP (none) -> M55342E12B10B0RT5
- R10, R11: MP (none) -> M55342K12B4E75RS2
- R3: MP (none) -> M55342K12B100ERS2
- R4: MP (none) -> M55342K12B20E0RS2
- R5: MP (none) -> 3386F-1-502TLF
- R6: MP (none) -> M55342K12B590DRS2
- R7: MP (none) -> M55342K12B56E2RWB
- R8, R9: MP (none) -> M55342K12B39E2RS2
- U10: MP (none) -> ADS1115IDGS
- U3: value ~ -> LILTGO touch
- U5: MP (none) -> TLV9001IDCKR
- U6: MP (none) -> MCP9808_MSOP
- U8: MP (none) -> DS3231MZ+
